Commit message: update

File: vehicle_urdf/urdf/vehicle.urdf.xacro (robot description, xacro)
@@ -7,5 +7,5 @@
     <visual>
       <geometry>
-        <box size="0.3 0.13 0.003"/>
+        <box size="0.2707 0.18 0.005"/>
       </geometry>
       <material name="blue"/>
@@ -13,5 +13,5 @@
     <collision>
       <geometry>
-        <box size="0.3 0.13 0.003"/>
+        <box size="0.2707 0.18 0.005"/>
       </geometry>
     </collision>
@@ -37,5 +37,5 @@
     <visual>
       <origin rpy="1.5708 0 0" xyz="0 0 0"/> <geometry>
-        <cylinder radius="0.045" length="0.04"/>
+        <cylinder radius="0.0325" length="0.033"/>
       </geometry>
       <material name="black"/>
@@ -44,5 +44,5 @@
       <origin rpy="1.5708 0 0" xyz="0 0 0"/>
       <geometry>
-        <cylinder radius="0.045" length="0.03"/>
+        <cylinder radius="0.0325" length="0.033"/>
       </geometry>
     </collision>
@@ -55,5 +55,5 @@
     <parent link="base_link"/>
     <child link="left_wheel"/>
-    <origin xyz="-0.1 0.09 -0.0165" rpy="0 0 0"/> <axis xyz="0 1 0"/>
+    <origin xyz="-0.10285 0.109 -0.0165" rpy="0 0 0"/> <axis xyz="0 1 0"/>
   </joint>
   <link name="right_wheel">
@@ -61,5 +61,5 @@
       <origin rpy="1.5708 0 0" xyz="0 0 0"/>
       <geometry>
-        <cylinder radius="0.045" length="0.04"/>
+        <cylinder radius="0.0325" length="0.033"/>
       </geometry>
       <material name="black"/>
@@ -68,5 +68,5 @@
       <origin rpy="1.5708 0 0" xyz="0 0 0"/>
       <geometry>
-        <cylinder radius="0.045" length="0.04"/>
+        <cylinder radius="0.0325" length="0.033"/>
       </geometry>
     </collision>
@@ -79,5 +79,5 @@
     <parent link="base_link"/>
     <child link="right_wheel"/>
-    <origin xyz="-0.1 -0.09 -0.0165" rpy="0 0 0"/> <axis xyz="0 1 0"/>
+    <origin xyz="-0.10285 -0.109 -0.0165" rpy="0 0 0"/> <axis xyz="0 1 0"/>
   </joint>
   <link name="caster_wheel">
@@ -90,5 +90,5 @@
     <collision>
       <geometry>
-        <sphere radius="0.03"/>
+        <sphere radius="0.025"/>
       </geometry>
     </collision>
@@ -102,4 +102,50 @@
     <child link="caster_wheel"/>
     <origin xyz="0.072 0 -0.0315" rpy="0 0 0"/>
+  </joint>
+    <link name="laser_cylinder_link">
+    <visual>
+      <origin rpy="0 0 0" xyz="0 0 0"/> <geometry>
+        <cylinder radius="0.008" length="0.066"/>
+      </geometry>
+      <material name="blue"/>
+    </visual>
+    <collision>
+      <origin rpy="0 0 0" xyz="0 0 0"/>
+      <geometry>
+        <cylinder radius="0.008" length="0.066"/>
+      </geometry>
+    </collision>
+    <inertial>
+      <mass value="0.5"/>
+      <inertia ixx="0.00037" ixy="0" ixz="0" iyy="0.00037" iyz="0" izz="0.000625"/>
+    </inertial>
+  </link>
+  <joint name="laser_cylinder_joint" type="fixed">
+    <parent link="base_link"/>
+    <child link="laser_cylinder_link"/>
+    <origin xyz="-0.01935 0 0.0355" rpy="0 0 0"/> <axis xyz="0 1 0"/>
+  </joint>
+      <link name="laser_link">
+    <visual>
+      <origin rpy="0 0 0" xyz="0 0 0"/> <geometry>
+        <cylinder radius="0.025" length="0.018"/>
+      </geometry>
+      <material name="black"/>
+    </visual>
+    <collision>
+      <origin rpy="0 0 0" xyz="0 0 0"/>
+      <geometry>
+        <cylinder radius="0.025" length="0.018"/>
+      </geometry>
+    </collision>
+    <inertial>
+      <mass value="0.5"/>
+      <inertia ixx="0.00037" ixy="0" ixz="0" iyy="0.00037" iyz="0" izz="0.000625"/>
+    </inertial>
+  </link>
+  <joint name="laser_joint" type="fixed">
+    <parent link="laser_cylinder_link"/>
+    <child link="laser_link"/>
+    <origin xyz="0 0 0.042" rpy="0 0 0"/> <axis xyz="0 1 0"/>
   </joint>
   <gazebo>
